Commit message: dsdq

File: src/rob_teleeop/rob_teleeop/urdf/base.urdf.xacro (robot description, xacro)
@@ -56,5 +56,5 @@
 <!-- Macro finger -->
 <xacro:finger parent="palm_link" prefix="finger1">
-<origin xyz="0.015141 -0.034337 0.105315" rpy="-241.826 96.5038 ${M_PI/2}" />
+<origin xyz="0.015141 -0.034337 0.105315" rpy="-241.826 96.5038 0.105315" />
 </xacro:finger>
 </robot>

File: src/rob_teleeop/rob_teleeop/urdf/finger.xacro (robot description, xacro)
@@ -2,5 +2,9 @@
 <robot xmlns:xacro="http://ros.org/wiki/xacro" name="finger">
 <xacro:macro name="finger" params="parent prefix joint_type">
-<link name="${prefix}_link" />
+<link name="${prefix}_link" >
+<visual>
+<mesh filename="file:///$(find robot_nano_hand_teleop)/models/robot_nano_hand_finger1_link1.stl" scale="1 1 1"/>
+</visual>
+</link>
 <joint name="${prefix}_joint" type="${joint_type}">
 <parent link="${parent}"/>

Commit message: d

File: src/rob_teleeop/rob_teleeop/urdf/base.urdf.xacro (robot description, xacro)
@@ -55,17 +55,17 @@
 </joint>
 <!-- Macro finger -->
-<xacro:finger parent="palm_link" prefix="finger1">
+<xacro:finger parent="palm_link" prefix="finger1" link="1">
 <origin xyz="0.015141 -0.034337 0.105315" rpy="-241.826 96.5038 0.105315" />
 </xacro:finger>
 </robot>
-<xacro:finger parent="palm_link" prefix="finger2">
+<xacro:finger parent="finger1" prefix="finger2" link="2">
 <origin xyz="-0.002487 0 0" rpy="9.00686 -0.124082 89.8118" />
 </xacro:finger>
 </robot>
-<xacro:finger parent="palm_link" prefix="finger3">
+<xacro:finger parent="finger2" prefix="finger3" link="3">
 <origin xyz="-0.040844 0.000126 0.00357" rpy="8.94359 0.091051 89.9831" />
 </xacro:finger>
 </robot>
-<xacro:finger parent="palm_link" prefix="finger4">
+<xacro:finger parent="finger3" prefix="finger4" link="4">
 <origin xyz="-0.029121 0.000013 0.002736" rpy="11.2847 -0.04374 89.947" />
 </xacro:finger>

File: src/rob_teleeop/rob_teleeop/urdf/finger.xacro (robot description, xacro)
@@ -1,8 +1,8 @@
 <?xml version="1.0"?>
 <robot xmlns:xacro="http://ros.org/wiki/xacro" name="finger">
-<xacro:macro name="finger" params="parent prefix joint_type">
+<xacro:macro name="finger" params="parent prefix joint_type link">
 <link name="${prefix}_link" >
 <visual>
-<mesh filename="file:///$(find robot_nano_hand_teleop)/models/robot_nano_hand_finger1_link1.stl" scale="1 1 1"/>
+<mesh filename="file:///$(find robot_nano_hand_teleop)/models/robot_nano_hand_finger1_link${link}.stl" scale="1 1 1"/>
 </visual>
 </link>

Commit message: qsd

File: src/rob_teleeop/rob_teleeop/urdf/base.urdf.xacro (robot description, xacro)
@@ -1,76 +1,73 @@
 <?xml version="1.0"?>
-<robot xmlns:xacro="http://www.ros.org/wiki/xacro" name="robot_nano_hand_teleop">
-<xacro:arg name="gazebo" default="false"/>
-<!-- Included URDF/XACRO Files -->
-<xacro:include filename="$(find robot_nano_hand_teleop)/urdf/finger.urdf.xacro" />
-<xacro:property name="M_PI" value="3.14159"/>
-<xacro:property name="baseMass" value="3.14159"/>
-<xacro:property name="baseLength" value="3.14159"/>
-<xacro:property name="baseWidth" value="3.14159"/>
-<xacro:property name="baseHeight" value="3.14159"/>
-<xacro:property name="chassisLength" value="3.14159"/>
-<xacro:property name="lower_limit" value="3.14159"/>
-<xacro:property name="upper_limit" value="3.14159"/>
-<link name="base_link">
-    <visual>
-    <origin xyz="0 0 0" rpy="0 0 0"/>
-    <geometry>
-    <mesh filename="file:///$(find robot_nano_hand_teleop)/models/robot_nano_hand_base.stl" scale="1 1 1"/>
-    </geometry>
-<!--         <material name="green"/> -->
-    </visual>
-    <collision>
-    <origin xyz="0 0 0" rpy="0 0 0"/>
-    <geometry>
-    <mesh filename="file:///$(find robot_nano_hand_teleop)/models/robot_nano_hand_base.stl" scale="1 1 1"/>
-    </geometry>
-    </collision>
-<!--     <inertial> -->
-<!--     <origin xyz="${-chassisLength/2 +0.2} 0 0.20" rpy="0 0 0"/> -->
-<!--     <mass value="${baseMass}"/> -->
-<!--     <xacro:box_inertia m="${baseMass}" x="${baseLength}"y="${baseWidth}" z="${baseHeight}"/> -->
-<!--     </inertial> -->
-</link>
-<!-- Palm link -->
-<link name="palm_link">
-    <visual>
-    <origin xyz="0 0 0" rpy="0 0 0"/>
-    <geometry>
-    <mesh filename="file:///$(find robot_nano_hand_teleop)/models/robot_nano_hand_palm.stl" scale="1 1 1"/>
-    </geometry>
-<!--    <material name="red"/> -->
-    </visual>
-    <collision>
-    <origin xyz="0 0 0.123" rpy="0 0 0"/>
-    <geometry>
-    <mesh filename="file:///$(find robot_nano_hand_teleop)/models/robot_nano_hand_palm.stl" scale="1 1 1"/>
-    </geometry>
-    </collision>
-<!--    <inertial> -->
-<!--    <origin xyz="${-chassisLength/2 +0.2} 0 0.20" rpy="0 0 0"/> -->
-<!--    <mass value="${baseMass}"/> -->
-<!--    <xacro:box_inertia m="${baseMass}" x="${baseLength}"y="${baseWidth}" z="${baseHeight}"/> -->
-<!--    </inertial> -->
-</link>
-<!-- Palm joint -->
-<joint name="my_joint" type="continuous">
-    <origin xyz="0 0 0.10" rpy="0 0 0" />
-    <parent link="base_link" />
-    <child link="palm_link" />
-    <limit effort="100" velocity="0"
-    lower="0" upper="12" />
-</joint>
-<!-- Macro finger -->
-<xacro:finger parent="palm_link" prefix="finger1" link="1" type="continuous">
-<origin xyz="0.015141 -0.034337 0.105315" rpy="-241.826 96.5038 0.105315" />
-</xacro:finger>
-<xacro:finger parent="finger1" prefix="finger2" link="2" type="continuous">
-<origin xyz="-0.002487 0 0" rpy="9.00686 -0.124082 89.8118" />
-</xacro:finger>
-<xacro:finger parent="finger2" prefix="finger3" link="3" type="continuous">
-<origin xyz="-0.040844 0.000126 0.00357" rpy="8.94359 0.091051 89.9831" />
-</xacro:finger>
-<xacro:finger parent="finger3" prefix="finger4" link="4" type="continuous">
-<origin xyz="-0.029121 0.000013 0.002736" rpy="11.2847 -0.04374 89.947" />
-</xacro:finger>
+<robot xmlns:xacro="http://www.ros.org/wiki/xacro" name="rob_teleeop">
+    <xacro:arg name="gazebo" default="false"/>
+    <xacro:include filename="$(find rob_teleeop)/rob_teleeop/urdf/finger.urdf.xacro" />
+    <xacro:property name="M_PI" value="3.14159"/>
+    <xacro:property name="baseMass" value="3.14159"/>
+    <xacro:property name="baseLength" value="3.14159"/>
+    <xacro:property name="baseWidth" value="3.14159"/>
+    <xacro:property name="baseHeight" value="3.14159"/>
+    <xacro:property name="chassisLength" value="3.14159"/>
+    <xacro:property name="lower_limit" value="3.14159"/>
+    <xacro:property name="upper_limit" value="3.14159"/>
+    <link name="base_link">
+        <visual>
+        <origin xyz="0 0 0" rpy="0 0 0"/>
+        <geometry>
+        <mesh filename="file:///$(find rob_teleeop)/models/robot_nano_hand_base.stl" scale="1 1 1"/>
+        </geometry>
+    <!--         <material name="green"/> -->
+        </visual>
+        <collision>
+        <origin xyz="0 0 0" rpy="0 0 0"/>
+        <geometry>
+        <mesh filename="file:///$(find rob_teleeop)/models/robot_nano_hand_base.stl" scale="1 1 1"/>
+        </geometry>
+        </collision>
+        <inertial>
+            <origin xyz="${-chassisLength/2 +0.2} 0 0.20" rpy="0 0 0"/>
+            <mass value="${baseMass}"/>
+            <xacro:box_inertia m="${baseMass}" x="${baseLength}"y="${baseWidth}" z="${baseHeight}"/>
+        </inertial>
+    </link>
+    <!-- Palm link -->
+    <link name="palm_link">
+        <visual>
+            <origin xyz="0 0 0" rpy="0 0 0"/>
+            <geometry>
+                <mesh filename="file:///$(find rob_teleeop)/models/robot_nano_hand_palm.stl" scale="1 1 1"/>
+            </geometry>
+        </visual>
+        <collision>
+            <origin xyz="0 0 0.123" rpy="0 0 0"/>
+            <geometry>
+                <mesh filename="file:///$(find rob_teleeop)/models/robot_nano_hand_palm.stl" scale="1 1 1"/>
+            </geometry>
+        </collision>
+    <!--    <inertial> -->
+    <!--    <origin xyz="${-chassisLength/2 +0.2} 0 0.20" rpy="0 0 0"/> -->
+    <!--    <mass value="${baseMass}"/> -->
+    <!--    <xacro:box_inertia m="${baseMass}" x="${baseLength}"y="${baseWidth}" z="${baseHeight}"/> -->
+    <!--    </inertial> -->
+    </link>
+    <!-- Palm joint -->
+    <joint name="my_joint" type="continuous">
+        <origin xyz="0 0 0.10" rpy="0 0 0" />
+        <parent link="base_link" />
+        <child link="palm_link" />
+        <limit effort="100" velocity="0" lower="0" upper="12" />
+    </joint>
+    <!-- Macro finger -->
+    <xacro:finger parent="palm_link" prefix="finger1" link="1" type="continuous">
+    <o  gin xyz="0.015141 -0.034337 0.105315" rpy="-241.826 96.5038 0.105315" />
+    </xacro:finger>
+    <xacro:finger parent="finger1" prefix="finger2" link="2" type="continuous">
+    <ori    in xyz="-0.002487 0 0" rpy="9.00686 -0.124082 89.8118" />
+    </xacro:finger>
+    <xacro:finger parent="finger2" prefix="finger3" link="3" type="continuous">
+    <or gin xyz="-0.040844 0.000126 0.00357" rpy="8.94359 0.091051 89.9831" />
+    </xacro:finger>
+    <xacro:finger parent="finger3" prefix="finger4" link="4" type="continuous">
+        rigin xyz="-0.029121 0.000013 0.002736" rpy="11.2847 -0.04374 89.947" />
+    </xacro:finger>
 </robot>

Commit message: qsd

File: src/rob_teleeop/rob_teleeop/urdf/base.urdf.xacro (robot description, xacro)
@@ -4,11 +4,4 @@
     <xacro:include filename="$(find rob_teleeop)/rob_teleeop/urdf/finger.urdf.xacro" />
     <xacro:property name="M_PI" value="3.14159"/>
-    <xacro:property name="baseMass" value="3.14159"/>
-    <xacro:property name="baseLength" value="3.14159"/>
-    <xacro:property name="baseWidth" value="3.14159"/>
-    <xacro:property name="baseHeight" value="3.14159"/>
-    <xacro:property name="chassisLength" value="3.14159"/>
-    <xacro:property name="lower_limit" value="3.14159"/>
-    <xacro:property name="upper_limit" value="3.14159"/>
     <link name="base_link">
         <visual>
@@ -60,14 +53,14 @@
     <!-- Macro finger -->
     <xacro:finger parent="palm_link" prefix="finger1" link="1" type="continuous">
-    <o  gin xyz="0.015141 -0.034337 0.105315" rpy="-241.826 96.5038 0.105315" />
+    <origin xyz="0.015141 -0.034337 0.105315" rpy="-241.826 96.5038 0.105315" />
     </xacro:finger>
     <xacro:finger parent="finger1" prefix="finger2" link="2" type="continuous">
-    <ori    in xyz="-0.002487 0 0" rpy="9.00686 -0.124082 89.8118" />
+    <origin xyz="-0.002487 0 0" rpy="9.00686 -0.124082 89.8118" />
     </xacro:finger>
     <xacro:finger parent="finger2" prefix="finger3" link="3" type="continuous">
-    <or gin xyz="-0.040844 0.000126 0.00357" rpy="8.94359 0.091051 89.9831" />
+    <origin xyz="-0.040844 0.000126 0.00357" rpy="8.94359 0.091051 89.9831" />
     </xacro:finger>
     <xacro:finger parent="finger3" prefix="finger4" link="4" type="continuous">
-        rigin xyz="-0.029121 0.000013 0.002736" rpy="11.2847 -0.04374 89.947" />
+     <origin xyz="-0.029121 0.000013 0.002736" rpy="11.2847 -0.04374 89.947" />
     </xacro:finger>
 </robot>

Commit message: qsd

File: src/rob_teleeop/rob_teleeop/urdf/base.urdf.xacro (robot description, xacro)
@@ -2,25 +2,20 @@
 <robot xmlns:xacro="http://www.ros.org/wiki/xacro" name="rob_teleeop">
     <xacro:arg name="gazebo" default="false"/>
-    <xacro:include filename="$(find rob_teleeop)/rob_teleeop/urdf/finger.urdf.xacro" />
+    <xacro:include filename="$(find rob_teleeop)/urdf/finger.urdf.xacro" />
     <xacro:property name="M_PI" value="3.14159"/>
     <link name="base_link">
         <visual>
-        <origin xyz="0 0 0" rpy="0 0 0"/>
-        <geometry>
-        <mesh filename="file:///$(find rob_teleeop)/models/robot_nano_hand_base.stl" scale="1 1 1"/>
-        </geometry>
-    <!--         <material name="green"/> -->
+            <origin xyz="0 0 0" rpy="0 0 0"/>
+            <geometry>
+                <mesh filename="file:///$(find rob_teleeop)/models/robot_nano_hand_base.stl" scale="1 1 1"/>
+            </geometry>
         </visual>
         <collision>
-        <origin xyz="0 0 0" rpy="0 0 0"/>
-        <geometry>
-        <mesh filename="file:///$(find rob_teleeop)/models/robot_nano_hand_base.stl" scale="1 1 1"/>
-        </geometry>
+            <origin xyz="0 0 0" rpy="0 0 0"/>
+            <geometry>
+                <mesh filename="file:///$(find rob_teleeop)/models/robot_nano_hand_base.stl" scale="1 1 1"/>
+            </geometry>
         </collision>
-        <inertial>
-            <origin xyz="${-chassisLength/2 +0.2} 0 0.20" rpy="0 0 0"/>
-            <mass value="${baseMass}"/>
-            <xacro:box_inertia m="${baseMass}" x="${baseLength}"y="${baseWidth}" z="${baseHeight}"/>
-        </inertial>
+        <!-- Add definition for all missing variable -->
     </link>
     <!-- Palm link -->
@@ -38,9 +33,4 @@
             </geometry>
         </collision>
-    <!--    <inertial> -->
-    <!--    <origin xyz="${-chassisLength/2 +0.2} 0 0.20" rpy="0 0 0"/> -->
-    <!--    <mass value="${baseMass}"/> -->
-    <!--    <xacro:box_inertia m="${baseMass}" x="${baseLength}"y="${baseWidth}" z="${baseHeight}"/> -->
-    <!--    </inertial> -->
     </link>
     <!-- Palm joint -->
@@ -52,15 +42,15 @@
     </joint>
     <!-- Macro finger -->
-    <xacro:finger parent="palm_link" prefix="finger1" link="1" type="continuous">
-    <origin xyz="0.015141 -0.034337 0.105315" rpy="-241.826 96.5038 0.105315" />
+    <xacro:finger parent="palm_link" prefix="finger1" link="1" joint_type="continuous">
+        <origin xyz="0.015141 -0.034337 0.105315" rpy="-241.826 96.5038 0.105315" />
     </xacro:finger>
-    <xacro:finger parent="finger1" prefix="finger2" link="2" type="continuous">
-    <origin xyz="-0.002487 0 0" rpy="9.00686 -0.124082 89.8118" />
+    <xacro:finger parent="finger1_link" prefix="finger2" link="2" joint_type="continuous">
+        <origin xyz="-0.002487 0 0" rpy="9.00686 -0.124082 89.8118" />
     </xacro:finger>
-    <xacro:finger parent="finger2" prefix="finger3" link="3" type="continuous">
-    <origin xyz="-0.040844 0.000126 0.00357" rpy="8.94359 0.091051 89.9831" />
+    <xacro:finger parent="finger2_link" prefix="finger3" link="3" joint_type="continuous">
+        <origin xyz="-0.040844 0.000126 0.00357" rpy="8.94359 0.091051 89.9831" />
     </xacro:finger>
-    <xacro:finger parent="finger3" prefix="finger4" link="4" type="continuous">
-     <origin xyz="-0.029121 0.000013 0.002736" rpy="11.2847 -0.04374 89.947" />
+    <xacro:finger parent="finger3_link" prefix="finger4" link="4" joint_type="continuous">
+        <origin xyz="-0.029121 0.000013 0.002736" rpy="11.2847 -0.04374 89.947" />
     </xacro:finger>
 </robot>

File: src/rob_teleeop/rob_teleeop/urdf/finger.urdf.xacro (robot description, xacro)
@@ -1,14 +1,16 @@
 <?xml version="1.0"?>
 <robot xmlns:xacro="http://ros.org/wiki/xacro" name="finger">
-<xacro:macro name="finger" params="parent prefix joint_type link">
-<link name="${prefix}_link" >
-<visual>
-<mesh filename="file:///$(find rob_teleeop)/models/robot_nano_hand_finger1_link${link}.stl" scale="1 1 1"/>
-</visual>
-</link>
-<joint name="${prefix}_joint" type="${joint_type}">
-<parent link="${parent}"/>
-<child link="${prefix}_link"/>
-</joint>
-</xacro:macro>
+    <xacro:macro name="finger" params="parent prefix link joint_type">
+        <link name="${prefix}_link" >
+            <visual>
+                <geometry>
+                    <mesh filename="file:///$(find rob_teleeop)/models/robot_nano_hand_finger1_link${link}.stl" scale="1 1 1"/>
+                </geometry>
+            </visual>
+        </link>
+        <joint name="${prefix}_joint" type="${joint_type}">
+            <parent link="${parent}"/>
+            <child link="${prefix}_link"/>
+        </joint>
+    </xacro:macro>
 </robot>

Commit message: qsdqs

File: src/rob_teleeop/rob_teleeop/urdf/base.urdf.xacro (robot description, xacro)
@@ -2,5 +2,5 @@
 <robot xmlns:xacro="http://www.ros.org/wiki/xacro" name="rob_teleeop">
     <xacro:arg name="gazebo" default="false"/>
-    <xacro:include filename="$(find rob_teleeop)/urdf/finger.urdf.xacro" />
+    <xacro:include filename="$(find rob_teleeop)/finger.urdf.xacro" />
     <xacro:property name="M_PI" value="3.14159"/>
     <link name="base_link">
@@ -8,5 +8,5 @@
             <origin xyz="0 0 0" rpy="0 0 0"/>
             <geometry>
-                <mesh filename="file:///$(find rob_teleeop)/models/robot_nano_hand_base.stl" scale="1 1 1"/>
+                <mesh filename="file:///$(find rob_teleeop)/robot_nano_hand_base.stl" scale="1 1 1"/>
             </geometry>
         </visual>
@@ -14,5 +14,5 @@
             <origin xyz="0 0 0" rpy="0 0 0"/>
             <geometry>
-                <mesh filename="file:///$(find rob_teleeop)/models/robot_nano_hand_base.stl" scale="1 1 1"/>
+                <mesh filename="file:///$(find rob_teleeop)/robot_nano_hand_base.stl" scale="1 1 1"/>
             </geometry>
         </collision>
@@ -24,5 +24,5 @@
             <origin xyz="0 0 0" rpy="0 0 0"/>
             <geometry>
-                <mesh filename="file:///$(find rob_teleeop)/models/robot_nano_hand_palm.stl" scale="1 1 1"/>
+                <mesh filename="file:///$(find rob_teleeop)/robot_nano_hand_palm.stl" scale="1 1 1"/>
             </geometry>
         </visual>
@@ -30,5 +30,5 @@
             <origin xyz="0 0 0.123" rpy="0 0 0"/>
             <geometry>
-                <mesh filename="file:///$(find rob_teleeop)/models/robot_nano_hand_palm.stl" scale="1 1 1"/>
+                <mesh filename="file:///$(find rob_teleeop)/robot_nano_hand_palm.stl" scale="1 1 1"/>
             </geometry>
         </collision>

Commit message: qsd

File: src/rob_teleeop/rob_teleeop/urdf/base.urdf.xacro (robot description, xacro)
@@ -42,15 +42,7 @@
     </joint>
     <!-- Macro finger -->
-    <xacro:finger parent="palm_link" prefix="finger1" link="1" joint_type="continuous">
-        <origin xyz="0.015141 -0.034337 0.105315" rpy="-241.826 96.5038 0.105315" />
-    </xacro:finger>
-    <xacro:finger parent="finger1_link" prefix="finger2" link="2" joint_type="continuous">
-        <origin xyz="-0.002487 0 0" rpy="9.00686 -0.124082 89.8118" />
-    </xacro:finger>
-    <xacro:finger parent="finger2_link" prefix="finger3" link="3" joint_type="continuous">
-        <origin xyz="-0.040844 0.000126 0.00357" rpy="8.94359 0.091051 89.9831" />
-    </xacro:finger>
-    <xacro:finger parent="finger3_link" prefix="finger4" link="4" joint_type="continuous">
-        <origin xyz="-0.029121 0.000013 0.002736" rpy="11.2847 -0.04374 89.947" />
-    </xacro:finger>
+    <xacro:finger parent="palm_link" prefix="finger1" link="1" joint_type="continuous" xyz="0.015141 -0.034337 0.105315" rpy="-241.826 96.5038 0.105315"/>
+    <xacro:finger parent="finger1_link" prefix="finger2" link="2" joint_type="continuous" xyz="-0.002487 0 0" rpy="9.00686 -0.124082 89.8118"/>
+    <xacro:finger parent="finger2_link" prefix="finger3" link="3" joint_type="continuous" xyz="-0.040844 0.000126 0.00357" rpy="8.94359 0.091051 89.9831"/>
+    <xacro:finger parent="finger3_link" prefix="finger4" link="4" joint_type="continuous" xyz="-0.029121 0.000013 0.002736" rpy="11.2847 -0.04374 89.947"/>
 </robot>

File: src/rob_teleeop/rob_teleeop/urdf/finger.urdf.xacro (robot description, xacro)
@@ -5,4 +5,5 @@
             <visual>
                 <geometry>
+                    <origin xyz="${xyz}" rpy="${rpy}" />
                     <mesh filename="file:///$(find rob_teleeop)/models/robot_nano_hand_finger1_link${link}.stl" scale="1 1 1"/>
                 </geometry>
@@ -10,4 +11,5 @@
         </link>
         <joint name="${prefix}_joint" type="${joint_type}">
+            <origin xyz="${xyz}" rpy="${rpy}" />
             <parent link="${parent}"/>
             <child link="${prefix}_link"/>

Commit message: qsd

File: src/rob_teleeop/rob_teleeop/urdf/base.urdf.xacro (robot description, xacro)
@@ -8,5 +8,5 @@
             <origin xyz="0 0 0" rpy="0 0 0"/>
             <geometry>
-                <mesh filename="file:///$(find rob_teleeop)/robot_nano_hand_base.stl" scale="1 1 1"/>
+                <mesh filename="$(find rob_teleeop)/robot_nano_hand_base.stl" scale="1 1 1"/>
             </geometry>
         </visual>

Commit message: qsd

File: src/rob_teleeop/rob_teleeop/urdf/base.urdf.xacro (robot description, xacro)
@@ -8,5 +8,5 @@
             <origin xyz="0 0 0" rpy="0 0 0"/>
             <geometry>
-                <mesh filename="$(find rob_teleeop)/robot_nano_hand_base.stl" scale="1 1 1"/>
+                <mesh filename="file:///$(find rob_teleeop)/robot_nano_hand_base.stl" scale="1 1 1"/>
             </geometry>
         </visual>

Commit message: qsd

File: src/rob_teleeop/rob_teleeop/urdf/base.urdf.xacro (robot description, xacro)
@@ -39,5 +39,5 @@
         <parent link="base_link" />
         <child link="palm_link" />
-        <limit effort="100" velocity="0" lower="0" upper="12" />
+        <limit effort="100" velocity="100" lower="0" upper="120" />
     </joint>
     <!-- Macro finger -->

Commit message: test add fixed join

File: src/rob_teleeop/rob_teleeop/urdf/base.urdf.xacro (robot description, xacro)
@@ -35,5 +35,5 @@
     </link>
     <!-- Palm joint -->
-    <joint name="my_joint" type="continuous">
+    <joint name="my_joint" type="fixed">
         <origin xyz="0 0 0.10" rpy="0 0 0" />
         <parent link="base_link" />
@@ -42,7 +42,7 @@
     </joint>
     <!-- Macro finger -->
-    <xacro:finger parent="palm_link" prefix="finger1" link="1" joint_type="continuous" xyz="0.015141 -0.034337 0.105315" rpy="-241.826 96.5038 0.105315"/>
-    <xacro:finger parent="finger1_link" prefix="finger2" link="2" joint_type="continuous" xyz="-0.002487 0 0" rpy="9.00686 -0.124082 89.8118"/>
-    <xacro:finger parent="finger2_link" prefix="finger3" link="3" joint_type="continuous" xyz="-0.040844 0.000126 0.00357" rpy="8.94359 0.091051 89.9831"/>
-    <xacro:finger parent="finger3_link" prefix="finger4" link="4" joint_type="continuous" xyz="-0.029121 0.000013 0.002736" rpy="11.2847 -0.04374 89.947"/>
+    <xacro:finger parent="palm_link" prefix="finger1" link="1" joint_type="fixed" xyz="0.015141 -0.034337 0.105315" rpy="-241.826 96.5038 0.105315"/>
+    <xacro:finger parent="finger1_link" prefix="finger2" link="2" joint_type="fixed" xyz="-0.002487 0 0" rpy="9.00686 -0.124082 89.8118"/>
+    <xacro:finger parent="finger2_link" prefix="finger3" link="3" joint_type="fixed" xyz="-0.040844 0.000126 0.00357" rpy="8.94359 0.091051 89.9831"/>
+    <xacro:finger parent="finger3_link" prefix="finger4" link="4" joint_type="fixed" xyz="-0.029121 0.000013 0.002736" rpy="11.2847 -0.04374 89.947"/>
 </robot>
