Commit message: sqd

File: src/rob_teleeop/rob_teleeop/urdf/base.urdf.xacro (robot description, xacro)
@@ -35,8 +35,9 @@
     </link>
     <!-- Palm joint -->
-    <joint name="my_joint" type="fixed">
+    <joint name="my_joint" type="revolut">
         <origin xyz="0 0 0.10" rpy="0 0 0" />
         <parent link="base_link" />
         <child link="palm_link" />
+        <axis xyz="1 0 0" />
         <limit effort="100" velocity="100" lower="0" upper="120" />
     </joint>

File: src/rob_teleeop/rob_teleeop/urdf/finger.urdf.xacro (robot description, xacro)
@@ -4,6 +4,6 @@
         <link name="${prefix}_link" >
             <visual>
+                <origin xyz="${xyz}" rpy="${rpy}" />
                 <geometry>
-                    <origin xyz="${xyz}" rpy="${rpy}" />
                     <mesh filename="file:///$(find rob_teleeop)/models/robot_nano_hand_finger1_link${link}.stl" scale="1 1 1"/>
                 </geometry>

Commit message: qsd

File: src/rob_teleeop/rob_teleeop/urdf/base.urdf.xacro (robot description, xacro)
@@ -35,5 +35,5 @@
     </link>
     <!-- Palm joint -->
-    <joint name="my_joint" type="revolut">
+    <joint name="my_joint" type="fixed">
         <origin xyz="0 0 0.10" rpy="0 0 0" />
         <parent link="base_link" />

Commit message: qsd

File: src/rob_teleeop/rob_teleeop/urdf/base.urdf.xacro (robot description, xacro)
@@ -35,5 +35,5 @@
     </link>
     <!-- Palm joint -->
-    <joint name="my_joint" type="fixed">
+    <joint name="my_joint" type="revolute">
         <origin xyz="0 0 0.10" rpy="0 0 0" />
         <parent link="base_link" />

Commit message: d

File: src/rob_teleeop/rob_teleeop/urdf/base.urdf.xacro (robot description, xacro)
@@ -36,9 +36,9 @@
     <!-- Palm joint -->
     <joint name="my_joint" type="revolute">
+        <axis xyz="1 0 0" />
+        <limit effort="0" velocity="0" lower="0" upper="50" />
         <origin xyz="0 0 0.10" rpy="0 0 0" />
         <parent link="base_link" />
         <child link="palm_link" />
-        <axis xyz="1 0 0" />
-        <limit effort="100" velocity="100" lower="0" upper="120" />
     </joint>
     <!-- Macro finger -->

Commit message: test

File: src/rob_teleeop/rob_teleeop/urdf/base.urdf.xacro (robot description, xacro)
@@ -6,5 +6,4 @@
     <link name="base_link">
         <visual>
-            <origin xyz="0 0 0" rpy="0 0 0"/>
             <geometry>
                 <mesh filename="file:///$(find rob_teleeop)/robot_nano_hand_base.stl" scale="1 1 1"/>

File: src/rob_teleeop/rob_teleeop/urdf/finger.urdf.xacro (robot description, xacro)
@@ -4,5 +4,5 @@
         <link name="${prefix}_link" >
             <visual>
-                <origin xyz="${xyz}" rpy="${rpy}" />
+                <origin xyz="0 0 0" rpy="0 0 0"/>
                 <geometry>
                     <mesh filename="file:///$(find rob_teleeop)/robot_nano_hand_finger1_link${link}.stl" scale="1 1 1"/>

Commit message: qsd

File: src/rob_teleeop/rob_teleeop/urdf/base.urdf.xacro (robot description, xacro)
@@ -34,5 +34,5 @@
     </link>
     <!-- Palm joint -->
-    <joint name="my_joint" type="revolute">
+    <joint name="my_joint" type="fixed">
         <axis xyz="1 0 0" />
         <limit effort="0" velocity="0" lower="0" upper="50" />

Commit message: test

File: src/rob_teleeop/rob_teleeop/urdf/base.urdf.xacro (robot description, xacro)
@@ -21,5 +21,5 @@
     <link name="palm_link">
         <visual>
-            <origin xyz="0 0 0" rpy="0 0 0"/>
+            <origin xyz="0 0 0.123" rpy="0 0 0"/>
             <geometry>
                 <mesh filename="file:///$(find rob_teleeop)/robot_nano_hand_palm.stl" scale="1 1 1"/>

Commit message: sqd

File: src/rob_teleeop/rob_teleeop/urdf/base.urdf.xacro (robot description, xacro)
@@ -34,5 +34,5 @@
     </link>
     <!-- Palm joint -->
-    <joint name="my_joint" type="fixed">
+    <joint name="my_joint" type="revolute">
         <axis xyz="1 0 0" />
         <limit effort="0" velocity="0" lower="0" upper="50" />

Commit message: qds

File: src/rob_teleeop/rob_teleeop/urdf/base.urdf.xacro (robot description, xacro)
@@ -34,5 +34,5 @@
     </link>
     <!-- Palm joint -->
-    <joint name="my_joint" type="revolute">
+    <joint name="handle_joint" type="revolute">
         <axis xyz="1 0 0" />
         <limit effort="0" velocity="0" lower="0" upper="50" />

Commit message: sqd

File: src/rob_teleeop/rob_teleeop/urdf/base.urdf.xacro (robot description, xacro)
@@ -21,5 +21,5 @@
     <link name="palm_link">
         <visual>
-            <origin xyz="0 0 0.123" rpy="0 0 0"/>
+            <origin xyz="0 0 0" rpy="0 0 0"/>
             <geometry>
                 <mesh filename="file:///$(find rob_teleeop)/robot_nano_hand_palm.stl" scale="1 1 1"/>

Commit message: qsd

File: src/rob_teleeop/rob_teleeop/urdf/base.urdf.xacro (robot description, xacro)
@@ -42,8 +42,8 @@
     </joint>
     <!-- Macro finger -->
-    <xacro:finger parent="palm_link" prefix="finger1" link="1" joint_type="fixed" xyz="0.015141 -0.034337 0.105315" rpy="${-241.826 / 360 * 2 * M_PI} ${96.5038 / 360 * 2 * M_PI} ${0.105315 / 360 * 2 * M_PI}"/>
+    <xacro:finger parent="palm_link" prefix="finger1" link="1" joint_type="fixed" xyz="0.015141 -0.034337 0.105315" rpy="${(-241.826 / 160) * M_PI} ${(96.5038 / 160) * M_PI} ${(0.105315 / 160) * M_PI}"/>
     same but rpy in radian using M_PI as pi and
-    <xacro:finger parent="finger1_link" prefix="finger2" link="2" joint_type="fixed" xyz="-0.002487 0 0" rpy="${9.00686 / 360 * 2 * M_PI} ${-0.124082 / 360 * 2 * M_PI} ${89.8118 / 360 * 2 * M_PI}"/>
-    <xacro:finger parent="finger2_link" prefix="finger3" link="3" joint_type="fixed" xyz="-0.040844 0.000126 0.00357" rpy="${8.94359 / 360 * 2 * M_PI} ${0.091051 / 360 * 2 * M_PI} ${89.9831 / 360 * 2 * M_PI}"/>
-    <xacro:finger parent="finger3_link" prefix="finger4" link="4" joint_type="fixed" xyz="-0.029121 0.000013 0.002736" rpy="${11.2847 / 360 * 2 * M_PI} ${-0.04374 / 360 * 2 * M_PI} ${89.947 / 360 * 2 * M_PI}"/>
+    <xacro:finger parent="finger1_link" prefix="finger2" link="2" joint_type="fixed" xyz="-0.002487 0 0" rpy="${(9.00686 / 160) * M_PI} ${(-0.124082 / 160) * M_PI} ${(89.8118 / 160) * M_PI}"/>
+    <xacro:finger parent="finger2_link" prefix="finger3" link="3" joint_type="fixed" xyz="-0.040844 0.000126 0.00357" rpy="${(8.94359 / 160) * M_PI} ${(0.091051 / 160) * M_PI} ${(89.9831 / 160) * M_PI}"/>
+    <xacro:finger parent="finger3_link" prefix="finger4" link="4" joint_type="fixed" xyz="-0.029121 0.000013 0.002736" rpy="${(11.2847 / 160) * M_PI} ${(-0.04374 / 160) * M_PI} ${(89.947 / 160) * M_PI}"/>
 </robot>

File: src/rob_teleeop/rob_teleeop/urdf/finger.urdf.xacro (robot description, xacro)
@@ -11,5 +11,5 @@
         </link>
         <joint name="${prefix}_joint" type="${joint_type}">
-            <origin xyz="0 0 0" rpy="0 0 0"/>
+            <origin xyz="${xyz}" rpy="${rpy}" />
             <parent link="${parent}"/>
             <child link="${prefix}_link"/>

Commit message: why

File: src/rob_teleeop/rob_teleeop/urdf/base.urdf.xacro (robot description, xacro)
@@ -6,4 +6,5 @@
     <link name="base_link">
         <visual>
+        <origin xyz="0 0 0" rpy="0 0 1.57"/>
             <geometry>
                 <mesh filename="file:///$(find rob_teleeop)/robot_nano_hand_base.stl" scale="1 1 1"/>
@@ -11,5 +12,5 @@
         </visual>
         <collision>
-            <origin xyz="0 0 0" rpy="0 0 0"/>
+            <origin xyz="0 0 0" rpy="0 0 1.57"/>
             <geometry>
                 <mesh filename="file:///$(find rob_teleeop)/robot_nano_hand_base.stl" scale="1 1 1"/>
@@ -21,5 +22,5 @@
     <link name="palm_link">
         <visual>
-            <origin xyz="0 0 0" rpy="0 0 0"/>
+            <origin xyz="0 0 0" rpy="0 0 1.57"/>
             <geometry>
                 <mesh filename="file:///$(find rob_teleeop)/robot_nano_hand_palm.stl" scale="1 1 1"/>
@@ -37,5 +38,5 @@
         <axis xyz="1 0 0" />
         <limit effort="0" velocity="0" lower="0" upper="50" />
-        <origin xyz="0 0 0.10" rpy="0 0 0" />
+        <origin xyz="0 0 0.132" rpy="0 0 0" />
         <parent link="base_link" />
         <child link="palm_link" />

File: src/rob_teleeop/rob_teleeop/urdf/finger.urdf.xacro (robot description, xacro)
@@ -4,5 +4,5 @@
         <link name="${prefix}_link" >
             <visual>
-                <origin xyz="0 0 0" rpy="0 0 0"/>
+                <origin xyz="0 0 0" rpy="0 0 1.57"/>
                 <geometry>
                     <mesh filename="file:///$(find rob_teleeop)/robot_nano_hand_finger1_link${link}.stl" scale="1 1 1"/>

Commit message: qsd

File: src/rob_teleeop/rob_teleeop/urdf/base.urdf.xacro (robot description, xacro)
@@ -6,5 +6,5 @@
     <link name="base_link">
         <visual>
-        <origin xyz="0 0 0" rpy="0 0 1.57"/>
+        <origin xyz="0 0 0" rpy="0 0 0"/>
             <geometry>
                 <mesh filename="file:///$(find rob_teleeop)/robot_nano_hand_base.stl" scale="1 1 1"/>
@@ -12,5 +12,5 @@
         </visual>
         <collision>
-            <origin xyz="0 0 0" rpy="0 0 1.57"/>
+            <origin xyz="0 0 0" rpy="0 0 0"/>
             <geometry>
                 <mesh filename="file:///$(find rob_teleeop)/robot_nano_hand_base.stl" scale="1 1 1"/>
@@ -22,5 +22,5 @@
     <link name="palm_link">
         <visual>
-            <origin xyz="0 0 0" rpy="0 0 1.57"/>
+            <origin xyz="0 0 0" rpy="0 0 0"/>
             <geometry>
                 <mesh filename="file:///$(find rob_teleeop)/robot_nano_hand_palm.stl" scale="1 1 1"/>

Commit message: ss

File: src/rob_teleeop/rob_teleeop/urdf/base.urdf.xacro (robot description, xacro)
@@ -6,5 +6,5 @@
     <link name="base_link">
         <visual>
-        <origin xyz="0 0 0" rpy="0 0 0"/>
+        <origin xyz="0 0 0" rpy="0 0 1.57"/>
             <geometry>
                 <mesh filename="file:///$(find rob_teleeop)/robot_nano_hand_base.stl" scale="1 1 1"/>
@@ -12,5 +12,5 @@
         </visual>
         <collision>
-            <origin xyz="0 0 0" rpy="0 0 0"/>
+            <origin xyz="0 0 0" rpy="0 0 1.57"/>
             <geometry>
                 <mesh filename="file:///$(find rob_teleeop)/robot_nano_hand_base.stl" scale="1 1 1"/>
@@ -22,5 +22,5 @@
     <link name="palm_link">
         <visual>
-            <origin xyz="0 0 0" rpy="0 0 0"/>
+            <origin xyz="0 0 0" rpy="0 0 1.57"/>
             <geometry>
                 <mesh filename="file:///$(find rob_teleeop)/robot_nano_hand_palm.stl" scale="1 1 1"/>
@@ -28,5 +28,5 @@
         </visual>
         <collision>
-            <origin xyz="0 0 0.123" rpy="0 0 0"/>
+            <origin xyz="0 0 0" rpy="0 0 1.57"/>
             <geometry>
                 <mesh filename="file:///$(find rob_teleeop)/robot_nano_hand_palm.stl" scale="1 1 1"/>
@@ -43,8 +43,8 @@
     </joint>
     <!-- Macro finger -->
-    <xacro:finger parent="palm_link" prefix="finger1" link="1" joint_type="fixed" xyz="0.015141 -0.034337 0.105315" rpy="-4.22 1.68 5.35"/>
+    <xacro:finger parent="palm_link" prefix="finger1" link="1" joint_type="fixed" xyz="0.015141 -0.034337 0.105315" rpy="-4.22 1.68 5.35" a="1.57"/>
     same but rpy in radian using M_PI as pi and
-    <xacro:finger parent="finger1_link" prefix="finger2" link="2" joint_type="fixed" xyz="-0.002487 0 0" rpy="0.157 -0.002 1.567"/>
-    <xacro:finger parent="finger2_link" prefix="finger3" link="3" joint_type="fixed" xyz="-0.040844 0.000126 0.00357" rpy="${(8.94359 / 160) * M_PI} ${(0.091051 / 160) * M_PI} ${(89.9831 / 160) * M_PI}"/>
-    <xacro:finger parent="finger3_link" prefix="finger4" link="4" joint_type="fixed" xyz="-0.029121 0.000013 0.002736" rpy="${(11.2847 / 160) * M_PI} ${(-0.04374 / 160) * M_PI} ${(89.947 / 160) * M_PI}"/>
+    <xacro:finger parent="finger1_link" prefix="finger2" link="2" joint_type="fixed" xyz="-0.002487 0 0" rpy="0.157 -0.002 1.567" a="0"/>
+    <xacro:finger parent="finger2_link" prefix="finger3" link="3" joint_type="fixed" xyz="-0.040844 0.000126 0.00357" rpy="${(8.94359 / 160) * M_PI} ${(0.091051 / 160) * M_PI} ${(89.9831 / 160) * M_PI}" a="0"/>
+    <xacro:finger parent="finger3_link" prefix="finger4" link="4" joint_type="fixed" xyz="-0.029121 0.000013 0.002736" rpy="${(11.2847 / 160) * M_PI} ${(-0.04374 / 160) * M_PI} ${(89.947 / 160) * M_PI}" a="0"/>
 </robot>

File: src/rob_teleeop/rob_teleeop/urdf/finger.urdf.xacro (robot description, xacro)
@@ -1,8 +1,8 @@
 <?xml version="1.0"?>
 <robot xmlns:xacro="http://ros.org/wiki/xacro" name="finger">
-    <xacro:macro name="finger" params="parent prefix link joint_type xyz rpy">
+    <xacro:macro name="finger" params="parent prefix link joint_type xyz rpy a">
         <link name="${prefix}_link" >
             <visual>
-                <origin xyz="0 0 0" rpy="0 0 0"/>
+                <origin xyz="0 0 0" rpy="0 0 ${a}"/>
                 <geometry>
                     <mesh filename="file:///$(find rob_teleeop)/robot_nano_hand_finger1_link${link}.stl" scale="1 1 1"/>

Commit message: qsd

File: src/rob_teleeop/rob_teleeop/urdf/base.urdf.xacro (robot description, xacro)
@@ -43,8 +43,8 @@
     </joint>
     <!-- Macro finger -->
-    <xacro:finger parent="palm_link" prefix="finger1" link="1" joint_type="fixed" xyz="0.015141 -0.034337 0.105315" rpy="-4.22 1.68 5.35" a="1.57"/>
+    <xacro:finger parent="palm_link" prefix="finger1" link="1" joint_type="fixed" xyz="0.015141 -0.034337 0.105315" rpy="-4.22 1.68 5.35"/>
     same but rpy in radian using M_PI as pi and
-    <xacro:finger parent="finger1_link" prefix="finger2" link="2" joint_type="fixed" xyz="-0.002487 0 0" rpy="0.157 -0.002 1.567" a="0"/>
-    <xacro:finger parent="finger2_link" prefix="finger3" link="3" joint_type="fixed" xyz="-0.040844 0.000126 0.00357" rpy="${(8.94359 / 160) * M_PI} ${(0.091051 / 160) * M_PI} ${(89.9831 / 160) * M_PI}" a="0"/>
-    <xacro:finger parent="finger3_link" prefix="finger4" link="4" joint_type="fixed" xyz="-0.029121 0.000013 0.002736" rpy="${(11.2847 / 160) * M_PI} ${(-0.04374 / 160) * M_PI} ${(89.947 / 160) * M_PI}" a="0"/>
+    <xacro:finger parent="finger1_link" prefix="finger2" link="2" joint_type="fixed" xyz="-0.002487 0 0" rpy="0.157 -0.002 1.567"/>
+    <xacro:finger parent="finger2_link" prefix="finger3" link="3" joint_type="fixed" xyz="-0.040844 0.000126 0.00357" rpy="${(8.94359 / 160) * M_PI} ${(0.091051 / 160) * M_PI} ${(89.9831 / 160) * M_PI}"/>
+    <xacro:finger parent="finger3_link" prefix="finger4" link="4" joint_type="fixed" xyz="-0.029121 0.000013 0.002736" rpy="${(11.2847 / 160) * M_PI} ${(-0.04374 / 160) * M_PI} ${(89.947 / 160) * M_PI}"/>
 </robot>

File: src/rob_teleeop/rob_teleeop/urdf/finger.urdf.xacro (robot description, xacro)
@@ -4,5 +4,5 @@
         <link name="${prefix}_link" >
             <visual>
-                <origin xyz="0 0 0" rpy="0 0 ${a}"/>
+                <origin xyz="0 0 0" rpy="0 0 1.57"/>
                 <geometry>
                     <mesh filename="file:///$(find rob_teleeop)/robot_nano_hand_finger1_link${link}.stl" scale="1 1 1"/>

Commit message: qds

File: src/rob_teleeop/rob_teleeop/urdf/base.urdf.xacro (robot description, xacro)
@@ -38,5 +38,5 @@
         <axis xyz="1 0 0" />
         <limit effort="0" velocity="0" lower="0" upper="50" />
-        <origin xyz="0 0 0.132" rpy="0 0 0" />
+        <origin xyz="0 0 0.10" rpy="0 0 0" />
         <parent link="base_link" />
         <child link="palm_link" />

Commit message: qsd

File: src/rob_teleeop/rob_teleeop/urdf/base.urdf.xacro (robot description, xacro)
@@ -6,5 +6,5 @@
     <link name="base_link">
         <visual>
-        <origin xyz="0 0 0" rpy="0 0 1.57"/>
+        <origin xyz="0 0 0" rpy="0 0 0"/>
             <geometry>
                 <mesh filename="file:///$(find rob_teleeop)/robot_nano_hand_base.stl" scale="1 1 1"/>

Commit message: qsd

File: src/rob_teleeop/rob_teleeop/urdf/base.urdf.xacro (robot description, xacro)
@@ -43,7 +43,7 @@
     </joint>
     <!-- Macro finger -->
-    <xacro:finger parent="palm_link" prefix="finger1" link="1" joint_type="fixed" xyz="0.015141 -0.034337 0.105315" rpy="-4.22 1.68 5.35"/>
+    <xacro:finger parent="palm_link" prefix="finger1" link="1" joint_type="fixed" xyz="0.015141 -0.034337 0.105315" rpy="-4.22 1.68 5.35" rot="0 0 1.57"/>
     same but rpy in radian using M_PI as pi and
-    <xacro:finger parent="finger1_link" prefix="finger2" link="2" joint_type="fixed" xyz="-0.002487 0 0" rpy="0.157 -0.002 1.567"/>
+    <xacro:finger parent="finger1_link" prefix="finger2" link="2" joint_type="fixed" xyz="-0.002487 0 0" rpy="0.157 -0.002 1.567" rot="${-1.57} 1.57 1.57"/>
     <xacro:finger parent="finger2_link" prefix="finger3" link="3" joint_type="fixed" xyz="-0.040844 0.000126 0.00357" rpy="${(8.94359 / 160) * M_PI} ${(0.091051 / 160) * M_PI} ${(89.9831 / 160) * M_PI}"/>
     <xacro:finger parent="finger3_link" prefix="finger4" link="4" joint_type="fixed" xyz="-0.029121 0.000013 0.002736" rpy="${(11.2847 / 160) * M_PI} ${(-0.04374 / 160) * M_PI} ${(89.947 / 160) * M_PI}"/>

File: src/rob_teleeop/rob_teleeop/urdf/finger.urdf.xacro (robot description, xacro)
@@ -1,8 +1,8 @@
 <?xml version="1.0"?>
 <robot xmlns:xacro="http://ros.org/wiki/xacro" name="finger">
-    <xacro:macro name="finger" params="parent prefix link joint_type xyz rpy">
+    <xacro:macro name="finger" params="parent prefix link joint_type xyz rpy rot">
         <link name="${prefix}_link" >
             <visual>
-                <origin xyz="0 0 0" rpy="0 0 1.57"/>
+                <origin xyz="0 0 0" rpy="${rot}"/>
                 <geometry>
                     <mesh filename="file:///$(find rob_teleeop)/robot_nano_hand_finger1_link${link}.stl" scale="1 1 1"/>

Commit message: qsd

File: src/rob_teleeop/rob_teleeop/urdf/base.urdf.xacro (robot description, xacro)
@@ -6,5 +6,5 @@
     <link name="base_link">
         <visual>
-        <origin xyz="0 0 0" rpy="0 0 0"/>
+        <origin xyz="0 0 0" rpy="0 0 1.57"/>
             <geometry>
                 <mesh filename="file:///$(find rob_teleeop)/robot_nano_hand_base.stl" scale="1 1 1"/>

Commit message: qsd

File: src/rob_teleeop/rob_teleeop/urdf/base.urdf.xacro (robot description, xacro)
@@ -36,5 +36,5 @@
     <!-- Palm joint -->
     <joint name="handle_joint" type="revolute">
-        <axis xyz="1 0 0" />
+        <axis xyz="0 1 0" />
         <limit effort="0" velocity="0" lower="0" upper="50" />
         <origin xyz="0 0 0.10" rpy="0 0 0" />

Commit message: qsd

File: src/rob_teleeop/rob_teleeop/urdf/base.urdf.xacro (robot description, xacro)
@@ -43,8 +43,7 @@
     </joint>
     <!-- Macro finger -->
-    <xacro:finger parent="palm_link" prefix="finger1" link="1" joint_type="fixed" xyz="0.015141 -0.034337 0.105315" rpy="-4.22 1.68 5.35" rot="0 0 1.57"/>
-    same but rpy in radian using M_PI as pi and
-    <xacro:finger parent="finger1_link" prefix="finger2" link="2" joint_type="fixed" xyz="-0.002487 0 0" rpy="${0.157} ${-0.002-1.57} 1.567" rot="0 -1.57 1.57"/>
-    <xacro:finger parent="finger2_link" prefix="finger3" link="3" joint_type="fixed" xyz="-0.040844 0.000126 0.00357" rpy="${(8.94359 / 160) * M_PI} ${(0.091051 / 160) * M_PI} ${(89.9831 / 160) * M_PI }" rot = "0 -1.57 1.57"/>
-    <xacro:finger parent="finger3_link" prefix="finger4" link="4" joint_type="fixed" xyz="-0.029121 0.000013 0.002736" rpy="${(11.2847 / 160) * M_PI} ${(-0.04374 / 160) * M_PI} ${(89.947 / 160) * M_PI}" rot="0 -1.57 1.57"/>
+    <xacro:finger parent="palm_link" prefix="finger1" link="1" joint_type="fixed" xyz="0.015141 -0.034337 0.105315" rpy="-4.22 1.68 5.35" rot="0 0 1.57" axis = "0 1 0"/>
+    <xacro:finger parent="finger1_link" prefix="finger2" link="2" joint_type="fixed" xyz="-0.002487 0 0" rpy="${0.157} ${-0.002-1.57} 1.567" rot="0 -1.57 1.57" axis = "0 0 1"/>
+    <xacro:finger parent="finger2_link" prefix="finger3" link="3" joint_type="fixed" xyz="-0.040844 0.000126 0.00357" rpy="${(8.94359 / 160) * M_PI} ${(0.091051 / 160) * M_PI} ${(89.9831 / 160) * M_PI }" rot = "0 -1.57 1.57" axis = "0 0 1"/>
+    <xacro:finger parent="finger3_link" prefix="finger4" link="4" joint_type="fixed" xyz="-0.029121 0.000013 0.002736" rpy="${(11.2847 / 160) * M_PI} ${(-0.04374 / 160) * M_PI} ${(89.947 / 160) * M_PI}" rot="0 -1.57 1.57" axis = "0 0 1"/>
 </robot>

File: src/rob_teleeop/rob_teleeop/urdf/finger.urdf.xacro (robot description, xacro)
@@ -1,5 +1,5 @@
 <?xml version="1.0"?>
 <robot xmlns:xacro="http://ros.org/wiki/xacro" name="finger">
-    <xacro:macro name="finger" params="parent prefix link joint_type xyz rpy rot">
+    <xacro:macro name="finger" params="parent prefix link joint_type xyz rpy rot axis">
         <link name="${prefix}_link" >
             <visual>
@@ -12,4 +12,5 @@
         <joint name="${prefix}_joint" type="${joint_type}">
             <origin xyz="${xyz}" rpy="${rpy}" />
+            <axis xyz="${axis}"/>
             <parent link="${parent}"/>
             <child link="${prefix}_link"/>
