Commit message: test macro a la macro

File: src/rob_teleeop/rob_teleeop/urdf/base.urdf.xacro (robot description, xacro)
@@ -2,5 +2,5 @@
 <robot xmlns:xacro="http://www.ros.org/wiki/xacro" name="rob_teleeop">
     <xacro:arg name="gazebo" default="false"/>
-    <xacro:include filename="$(find rob_teleeop)/finger.urdf.xacro" />
+    <xacro:include filename="$(find rob_teleeop)/ff.urdf.xacro" />
     <xacro:property name="M_PI" value="3.14159"/>
     <link name="base_link">
@@ -43,7 +43,4 @@
     </joint>
     <!-- Macro finger -->
-    <xacro:finger parent="palm_link" prefix="finger1" link="1" joint_type="revolute" xyz="0.015141 -0.034337 0.105315" rpy="-4.22 1.68 5.35" rot="0 0 1.57" axis = "1 0 0"/>
-    <xacro:finger parent="finger1_link" prefix="finger2" link="2" joint_type="revolute" xyz="-0.002487 0 0" rpy="${0.157} ${-0.002-1.57} 1.567" rot="0 -1.57 1.57" axis = "0 0 1"/>
-    <xacro:finger parent="finger2_link" prefix="finger3" link="3" joint_type="revolute" xyz="-0.040844 0.000126 0.00357" rpy="${(8.94359 / 160) * M_PI} ${(0.091051 / 160) * M_PI} ${(89.9831 / 160) * M_PI }" rot = "0 -1.57 1.57" axis = "0 0 1"/>
-    <xacro:finger parent="finger3_link" prefix="finger4" link="4" joint_type="revolute" xyz="-0.029121 0.000013 0.002736" rpy="${(11.2847 / 160) * M_PI} ${(-0.04374 / 160) * M_PI} ${(89.947 / 160) * M_PI}" rot="0 -1.57 1.57" axis = "0 0 1"/>
+ <xacro:ff base_ref="palm_link" nb="1"/>
 </robot>

File: src/rob_teleeop/rob_teleeop/urdf/finger.urdf.xacro (robot description, xacro)
@@ -1,19 +1,19 @@
 <?xml version="1.0"?>
 <robot xmlns:xacro="http://ros.org/wiki/xacro" name="finger">
-    <xacro:macro name="finger" params="parent prefix link joint_type xyz rpy rot axis">
-        <link name="${prefix}_link" >
+    <xacro:macro name="finger" params="parent nb prefix link joint_type xyz rpy rot axis">
+        <link name="finger${nb}_link{link}" >
             <visual>
                 <origin xyz="0 0 0" rpy="${rot}"/>
                 <geometry>
-                    <mesh filename="file:///$(find rob_teleeop)/robot_nano_hand_finger1_link${link}.stl" scale="1 1 1"/>
+                    <mesh filename="file:///$(find rob_teleeop)/robot_nano_hand_finger${nb}_link${link}.stl" scale="1 1 1"/>
                 </geometry>
             </visual>
         </link>
-        <joint name="${prefix}_joint" type="${joint_type}">
+        <joint name="finger${nb}_joint{link}" type="${joint_type}">
             <origin xyz="${xyz}" rpy="${rpy}" />
             <axis xyz="${axis}"/>
             <limit effort="0" velocity="0" lower="-100" upper="100" />
             <parent link="${parent}"/>
-            <child link="${prefix}_link"/>
+            <child link="finger${nb}_link{link}"/>
         </joint>
     </xacro:macro>

Commit message: qsd

File: src/rob_teleeop/rob_teleeop/urdf/base.urdf.xacro (robot description, xacro)
@@ -6,5 +6,5 @@
     <link name="base_link">
         <visual>
-        <origin xyz="0 0 0" rpy="0 0 1.57"/>
+        <origin xyz="0 0 0" rpy="0 0 0"/>
             <geometry>
                 <mesh filename="file:///$(find rob_teleeop)/robot_nano_hand_base.stl" scale="1 1 1"/>
@@ -12,5 +12,5 @@
         </visual>
         <collision>
-            <origin xyz="0 0 0" rpy="0 0 1.57"/>
+            <origin xyz="0 0 0" rpy="0 0 0"/>
             <geometry>
                 <mesh filename="file:///$(find rob_teleeop)/robot_nano_hand_base.stl" scale="1 1 1"/>
@@ -22,5 +22,5 @@
     <link name="palm_link">
         <visual>
-            <origin xyz="0 0 0" rpy="0 0 1.57"/>
+            <origin xyz="0 0 0.132" rpy="0 0 0"/>
             <geometry>
                 <mesh filename="file:///$(find rob_teleeop)/robot_nano_hand_palm.stl" scale="1 1 1"/>
@@ -28,5 +28,5 @@
         </visual>
         <collision>
-            <origin xyz="0 0 0" rpy="0 0 1.57"/>
+            <origin xyz="0 0 0" rpy="0 0 0"/>
             <geometry>
                 <mesh filename="file:///$(find rob_teleeop)/robot_nano_hand_palm.stl" scale="1 1 1"/>
@@ -36,5 +36,5 @@
     <!-- Palm joint -->
     <joint name="handle_joint" type="revolute">
-        <axis xyz="0 1 0" />
+        <axis xyz="1 0 0" />
         <limit effort="0" velocity="0" lower="0" upper="50" />
         <origin xyz="0 0 0.10" rpy="0 0 0" />

File: src/rob_teleeop/rob_teleeop/urdf/ff.urdf.xacro (robot description, xacro)
@@ -8,7 +8,7 @@
     <!--    <xacro:finger parent="finger${nb}_link3" nb="${nb}" link="4" joint_type="revolute" xyz="-0.029121 0.000013 0.002736" rpy="${(11.2847 / 160) * M_PI} ${(-0.04374 / 160) * M_PI} ${(89.947 / 160) * M_PI}" rot="0 -1.57 1.57" axis = "0 0 1"/> -->
         <xacro:finger parent="${base_ref}" nb="${nb}" link="1" joint_type="revolute" xyz="0.015141 -0.034337 0.105315" rpy="-4.22 1.68 5.35" rot="0 0 0" axis = "1 0 0"/>
-        <xacro:finger parent="finger${nb}_link1" nb="${nb}" link="2" joint_type="revolute" xyz="-0.002487 0 0" rpy="0 0 0" rot="0 0 0" axis = "0 0 1"/>
-        <xacro:finger parent="finger${nb}_link2" nb="${nb}" link="3" joint_type="revolute" xyz="-0.040844 0.000126 0.00357" rpy="0 0 0" rot = "0 0 0" axis = "0 0 1"/>
-        <xacro:finger parent="finger${nb}_link3" nb="${nb}" link="4" joint_type="revolute" xyz="-0.029121 0.000013 0.002736" rpy="0 0 0" rot="0 0 0" axis = "0 0 1"/>
+        <xacro:finger parent="finger${nb}_link1" nb="${nb}" link="2" joint_type="revolute" xyz="0 -0.172006 0.127457" rpy="0 0 0" rot="0 0 0" axis = "0 0 1"/>
+        <xacro:finger parent="finger${nb}_link2" nb="${nb}" link="3" joint_type="revolute" xyz="0 -0.172005 0.130058" rpy="0 0 0" rot = "0 0 0" axis = "0 0 1"/>
+        <xacro:finger parent="finger${nb}_link3" nb="${nb}" link="4" joint_type="revolute" xyz="0.006306 -0.171866 0.200022" rpy="0 0 0" rot="0 0 0" axis = "0 0 1"/>
     </xacro:macro>
 </robot>

Commit message: qsd

File: src/rob_teleeop/rob_teleeop/urdf/base.urdf.xacro (robot description, xacro)
@@ -22,5 +22,5 @@
     <link name="palm_link">
         <visual>
-            <origin xyz="0 0 0.132" rpy="0 0 0"/>
+            <origin xyz="0 0 0" rpy="0 0 0"/>
             <geometry>
                 <mesh filename="file:///$(find rob_teleeop)/robot_nano_hand_palm.stl" scale="1 1 1"/>

Commit message: qsd

File: src/rob_teleeop/rob_teleeop/urdf/base.urdf.xacro (robot description, xacro)
@@ -38,5 +38,5 @@
         <axis xyz="1 0 0" />
         <limit effort="0" velocity="0" lower="0" upper="50" />
-        <origin xyz="0 0 0.10" rpy="0 0 0" />
+        <origin xyz="0 0 0.132" rpy="0 0 0" />
         <parent link="base_link" />
         <child link="palm_link" />

Commit message: s

File: src/rob_teleeop/rob_teleeop/urdf/base.urdf.xacro (robot description, xacro)
@@ -43,4 +43,5 @@
     </joint>
     <!-- Macro finger -->
- <xacro:ff base_ref="palm_link" nb="1"/>
+ <xacro:ff base_ref="palm_link" nb="1" p1="0 0.02 0.02" p2="0 0 0.02" p3="0 0 0.02" p4= "0 0 0.02"/>
+ <xacro:ff base_ref="palm_link" nb="2" p1="0 -0.02 0.02" p2="0 0 0.02" p3="0 0 0.02" p4= "0 0 0.02"/>
 </robot>

File: src/rob_teleeop/rob_teleeop/urdf/ff.urdf.xacro (robot description, xacro)
@@ -2,13 +2,13 @@
 <robot xmlns:xacro="http://ros.org/wiki/xacro" name="rob_teleeop">
     <xacro:include filename="$(find rob_teleeop)/finger.urdf.xacro" />
-    <xacro:macro name="ff" params="base_ref nb">
+    <xacro:macro name="ff" params="base_ref nb p1 p2 p3 p4">
     <!--    <xacro:finger parent="${base_ref}" nb="${nb}" link="1" joint_type="revolute" xyz="0.015141 -0.034337 0.105315" rpy="-4.22 1.68 5.35" rot="0 0 1.57" axis = "1 0 0"/> -->
     <!--    <xacro:finger parent="finger${nb}_link1" nb="${nb}" link="2" joint_type="revolute" xyz="-0.002487 0 0" rpy="${0.157} ${-0.002-1.57} 1.567" rot="0 -1.57 1.57" axis = "0 0 1"/> -->
     <!--    <xacro:finger parent="finger${nb}_link2" nb="${nb}" link="3" joint_type="revolute" xyz="-0.040844 0.000126 0.00357" rpy="${(8.94359 / 160) * M_PI} ${(0.091051 / 160) * M_PI} ${(89.9831 / 160) * M_PI }" rot = "0 -1.57 1.57" axis = "0 0 1"/> -->
     <!--    <xacro:finger parent="finger${nb}_link3" nb="${nb}" link="4" joint_type="revolute" xyz="-0.029121 0.000013 0.002736" rpy="${(11.2847 / 160) * M_PI} ${(-0.04374 / 160) * M_PI} ${(89.947 / 160) * M_PI}" rot="0 -1.57 1.57" axis = "0 0 1"/> -->
-        <xacro:finger parent="${base_ref}" nb="${nb}" link="1" joint_type="revolute" xyz="0.02 0 0.2" rpy="0 0 0" rot="0 0 0" axis = "1 0 0"/>
-        <xacro:finger parent="finger${nb}_link1" nb="${nb}" link="2" joint_type="revolute" xyz="0 0 0.02" rpy="0 0 0" rot="0 0 0" axis = "0 0 1"/>
-        <xacro:finger parent="finger${nb}_link2" nb="${nb}" link="3" joint_type="revolute" xyz="0 0 0.02" rpy="0 0 0" rot = "0 0 0" axis = "0 0 1"/>
-        <xacro:finger parent="finger${nb}_link3" nb="${nb}" link="4" joint_type="revolute" xyz="0 0 0.02" rpy="0 0 0" rot="0 0 0" axis = "0 0 1"/>
+        <xacro:finger parent="${base_ref}" nb="${nb}" link="1" joint_type="revolute" xyz="${p1}" rpy="0 0 0" rot="0 0 0" axis = "1 0 0"/>
+        <xacro:finger parent="finger${nb}_link1" nb="${nb}" link="2" joint_type="revolute" xyz="${p2}" rpy="0 0 0" rot="0 0 0" axis = "0 0 1"/>
+        <xacro:finger parent="finger${nb}_link2" nb="${nb}" link="3" joint_type="revolute" xyz="${p3}" rpy="0 0 0" rot = "0 0 0" axis = "0 0 1"/>
+        <xacro:finger parent="finger${nb}_link3" nb="${nb}" link="4" joint_type="revolute" xyz="${p4}" rpy="0 0 0" rot="0 0 0" axis = "0 0 1"/>
     </xacro:macro>
 </robot>

Commit message: qsd

File: src/rob_teleeop/rob_teleeop/urdf/base.urdf.xacro (robot description, xacro)
@@ -22,5 +22,5 @@
     <link name="palm_link">
         <visual>
-            <origin xyz="0 0 0" rpy="0 0 0"/>
+            <origin xyz="0 0 0.132" rpy="0 0 0"/>
             <geometry>
                 <mesh filename="file:///$(find rob_teleeop)/robot_nano_hand_palm.stl" scale="1 1 1"/>
@@ -38,10 +38,10 @@
         <axis xyz="1 0 0" />
         <limit effort="0" velocity="0" lower="0" upper="50" />
-        <origin xyz="0 0 0.132" rpy="0 0 0" />
+        <origin xyz="0 0 0.10" rpy="0 0 0" />
         <parent link="base_link" />
         <child link="palm_link" />
     </joint>
     <!-- Macro finger -->
- <xacro:ff base_ref="palm_link" nb="1" p1="0 -0.01 0.15" p2="0 0 0.0026" p3="0.00357 0.000126 0.000126" p4= "0.006306 0.000139 0.029247"/>
+ <xacro:ff base_ref="palm_link" nb="1" p1="0 -0.01 0.15" p2="0 0 0.0026" p3="0.00357 0.000126 0.000126" p4="0.006306 0.000139 0.029247"/>
  <xacro:ff base_ref="palm_link" nb="2" p1="0 0.2 0.02" p2="0 0 0.02" p3="0 0 0.02" p4= "0 0 0.02"/>
 </robot>

Commit message: sd

File: src/rob_teleeop/rob_teleeop/urdf/base.urdf.xacro (robot description, xacro)
@@ -43,5 +43,6 @@
     </joint>
     <!-- Macro finger -->
- <xacro:ff base_ref="palm_link" nb="1" p1="0 -0.01 0.15" p2="0 0 0.0026" p3="0.00357 0.000126 0.000126" p4="0.006306 0.000139 0.029247"/>
- <xacro:ff base_ref="palm_link" nb="2" p1="0 0.2 0.02" p2="0 0 0.02" p3="0 0 0.02" p4= "0 0 0.02"/>
+ <xacro:ff base_ref="palm_link" nb="1"
+ r1="0.134884 0.077146 0.149703" p1="0.014588 -0.034298 0.105371" p2="0 0 0.0026" p3="0.00357 0.000126 0.040844" p4="0.006306 0.000139 0.029247"/>
+ <xacro:ff base_ref="palm_link" nb="2" r1="" p1="0 0.2 0.02" p2="0 0 0.02" p3="0 0 0.02" p4= "0 0 0.02"/>
 </robot>

File: src/rob_teleeop/rob_teleeop/urdf/ff.urdf.xacro (robot description, xacro)
@@ -2,10 +2,10 @@
 <robot xmlns:xacro="http://ros.org/wiki/xacro" name="rob_teleeop">
     <xacro:include filename="$(find rob_teleeop)/finger.urdf.xacro" />
-    <xacro:macro name="ff" params="base_ref nb p1 p2 p3 p4">
+    <xacro:macro name="ff" params="base_ref nb r1 p1 p2 p3 p4">
     <!--    <xacro:finger parent="${base_ref}" nb="${nb}" link="1" joint_type="revolute" xyz="0.015141 -0.034337 0.105315" rpy="-4.22 1.68 5.35" rot="0 0 1.57" axis = "1 0 0"/> -->
     <!--    <xacro:finger parent="finger${nb}_link1" nb="${nb}" link="2" joint_type="revolute" xyz="-0.002487 0 0" rpy="${0.157} ${-0.002-1.57} 1.567" rot="0 -1.57 1.57" axis = "0 0 1"/> -->
     <!--    <xacro:finger parent="finger${nb}_link2" nb="${nb}" link="3" joint_type="revolute" xyz="-0.040844 0.000126 0.00357" rpy="${(8.94359 / 160) * M_PI} ${(0.091051 / 160) * M_PI} ${(89.9831 / 160) * M_PI }" rot = "0 -1.57 1.57" axis = "0 0 1"/> -->
     <!--    <xacro:finger parent="finger${nb}_link3" nb="${nb}" link="4" joint_type="revolute" xyz="-0.029121 0.000013 0.002736" rpy="${(11.2847 / 160) * M_PI} ${(-0.04374 / 160) * M_PI} ${(89.947 / 160) * M_PI}" rot="0 -1.57 1.57" axis = "0 0 1"/> -->
-        <xacro:finger parent="${base_ref}" nb="${nb}" link="1" joint_type="revolute" xyz="${p1}" rpy="0 0 0" rot="0 0 0" axis = "1 0 0"/>
+        <xacro:finger parent="${base_ref}" nb="${nb}" link="1" joint_type="revolute" xyz="${p1}" rpy="${r1}" rot="0 0 0" axis = "1 0 0"/>
         <xacro:finger parent="finger${nb}_link1" nb="${nb}" link="2" joint_type="revolute" xyz="${p2}" rpy="0 0 0" rot="0 0 0" axis = "0 0 1"/>
         <xacro:finger parent="finger${nb}_link2" nb="${nb}" link="3" joint_type="revolute" xyz="${p3}" rpy="0 0 0" rot = "0 0 0" axis = "0 0 1"/>

Commit message: qsd

File: src/rob_teleeop/rob_teleeop/urdf/base.urdf.xacro (robot description, xacro)
@@ -22,5 +22,5 @@
     <link name="palm_link">
         <visual>
-            <origin xyz="0 0 0.132" rpy="0 0 0"/>
+            <origin xyz="0 0 0" rpy="0 0 0"/>
             <geometry>
                 <mesh filename="file:///$(find rob_teleeop)/robot_nano_hand_palm.stl" scale="1 1 1"/>
@@ -43,6 +43,5 @@
     </joint>
     <!-- Macro finger -->
- <xacro:ff base_ref="palm_link" nb="1"
- r1="0.134884 0.077146 0.149703" p1="0.014588 -0.034298 0.105371" p2="0 0 0.0026" p3="0.00357 0.000126 0.040844" p4="0.006306 0.000139 0.029247"/>
- <xacro:ff base_ref="palm_link" nb="2" r1="" p1="0 0.2 0.02" p2="0 0 0.02" p3="0 0 0.02" p4= "0 0 0.02"/>
+ <xacro:ff base_ref="palm_link" nb="1" r1="0.134884 0.077146 0.149703" p1="0.014588 -0.034298 0.105371" p2="0 0 0.0026" p3="0.00357 0.000126 0.040844" p4="0.006306 0.000139 0.029247"/>
+ <xacro:ff base_ref="palm_link" nb="2" r1="0.062643 -0.000111 0.073654" p1="0.007772 -0.013612 0.117984" p2="0 0 0.0026" p3="-0.003183 0 0.045388" p4="-0.002027 0 0.032436"/>
 </robot>

Commit message: ss

File: src/rob_teleeop/rob_teleeop/urdf/base.urdf.xacro (robot description, xacro)
@@ -6,5 +6,5 @@
     <link name="base_link">
         <visual>
-        <origin xyz="0 0 0" rpy="0 0 0"/>
+        <origin xyz="0 0 0" rpy="0 0 1.57"/>
             <geometry>
                 <mesh filename="file:///$(find rob_teleeop)/robot_nano_hand_base.stl" scale="1 1 1"/>
@@ -22,5 +22,5 @@
     <link name="palm_link">
         <visual>
-            <origin xyz="0 0 0" rpy="0 0 0"/>
+            <origin xyz="0 0 0" rpy="0 0 1.57"/>
             <geometry>
                 <mesh filename="file:///$(find rob_teleeop)/robot_nano_hand_palm.stl" scale="1 1 1"/>

Commit message: qsd

File: src/rob_teleeop/rob_teleeop/urdf/base.urdf.xacro (robot description, xacro)
@@ -1,4 +1,10 @@
 <?xml version="1.0"?>
 <robot xmlns:xacro="http://www.ros.org/wiki/xacro" name="rob_teleeop">
+  <material name="blue">
+    <color rgba="0 0 0.8 1"/>
+  </material>
+  <material name="white">
+    <color rgba="1 1 1 1"/>
+  </material>
     <xacro:arg name="gazebo" default="false"/>
     <xacro:include filename="$(find rob_teleeop)/ff.urdf.xacro" />
@@ -10,4 +16,5 @@
                 <mesh filename="file:///$(find rob_teleeop)/robot_nano_hand_base.stl" scale="1 1 1"/>
             </geometry>
+        <material name="blue"/>
         </visual>
         <collision>
@@ -26,4 +33,5 @@
                 <mesh filename="file:///$(find rob_teleeop)/robot_nano_hand_palm.stl" scale="1 1 1"/>
             </geometry>
+            <material name="white"/>
         </visual>
         <collision>

Commit message: qsdqs

File: src/rob_teleeop/rob_teleeop/urdf/base.urdf.xacro (robot description, xacro)
@@ -19,5 +19,5 @@
         </visual>
         <collision>
-            <origin xyz="0 0 0" rpy="0 0 0"/>
+            <origin xyz="0 0 0" rpy="0 0 1.57"/>
             <geometry>
                 <mesh filename="file:///$(find rob_teleeop)/robot_nano_hand_base.stl" scale="1 1 1"/>
@@ -36,5 +36,5 @@
         </visual>
         <collision>
-            <origin xyz="0 0 0" rpy="0 0 0"/>
+            <origin xyz="0 0 0" rpy="0 0 1.57"/>
             <geometry>
                 <mesh filename="file:///$(find rob_teleeop)/robot_nano_hand_palm.stl" scale="1 1 1"/>
@@ -51,6 +51,18 @@
     </joint>
     <!-- Macro finger -->
- <xacro:ff base_ref="palm_link" nb="1" r1="0.134884 0.077146 0.149703" p1="0.014588 -0.034298 0.105371" p2="0 0 0.0026" p3="0.00357 0.000126 0.040844" p4="0.006306 0.000139 0.029247" axis="0 1 0"/>
- <xacro:ff base_ref="palm_link" nb="2" r1="0.062643 -0.000111 0.073654" p1="0.007772 -0.013612 0.117984" p2="0 0 0.0026" p3="-0.003183 0 0.045388" p4="-0.002027 0 0.032436" axis="0 1 0"/>
+ <xacro:ff base_ref="palm_link" nb="1"
+    r1="0.134884 0.077146 0.149703"
+    p1="0.014588 -0.034298 0.105371"
+    p2="0 0 0.0026"
+    p3="0.00357 0.000126 0.040844"
+    p4="0.006306 0.000139 0.029247"
+    axis="0 1 0"/>
+ <xacro:ff base_ref="palm_link" nb="2"
+    r1="0.062643 -0.000111 0.073654"
+    p1="0.007772 -0.013612 0.117984"
+    p2="0 0 0.0026"
+    p3="-0.003183 0 0.045388"
+    p4="-0.002027 0 0.032436"
+    axis="0 1 0"/>
 <xacro:ff base_ref="palm_link" nb="3"
     r1="0 -0.014913 0"

File: src/rob_teleeop/rob_teleeop/urdf/finger.urdf.xacro (robot description, xacro)
@@ -9,4 +9,10 @@
                 </geometry>
             </visual>
+            <collision>
+            <origin xyz="0 0 0" rpy="${rot}"/>
+            <geometry>
+                <mesh filename="file:///$(find rob_teleeop)/robot_nano_hand_finger${nb}_link${link}.stl" scale="1 1 1"/>
+            </geometry>
+        </collision>
         </link>
         <joint name="finger${nb}_joint${link}" type="${joint_type}">
