Commit message: qsd

File: src/rob_teleeop/rob_teleeop/urdf/finger.urdf.xacro (robot description, xacro)
@@ -4,5 +4,5 @@
 <link name="${prefix}_link" >
 <visual>
-<mesh filename="file:///$(find robot_nano_hand_teleop)/models/robot_nano_hand_finger1_link${link}.stl" scale="1 1 1"/>
+<mesh filename="file:///$(find rob_teleeop)/models/robot_nano_hand_finger1_link${link}.stl" scale="1 1 1"/>
 </visual>
 </link>

Commit message: qsd

File: src/rob_teleeop/rob_teleeop/urdf/finger.urdf.xacro (robot description, xacro)
@@ -1,5 +1,5 @@
 <?xml version="1.0"?>
 <robot xmlns:xacro="http://ros.org/wiki/xacro" name="finger">
-    <xacro:macro name="finger" params="parent prefix link joint_type">
+    <xacro:macro name="finger" params="parent prefix link joint_type xyz rpy">
         <link name="${prefix}_link" >
             <visual>

Commit message: sdq

File: src/rob_teleeop/rob_teleeop/urdf/finger.urdf.xacro (robot description, xacro)
@@ -6,5 +6,5 @@
                 <origin xyz="${xyz}" rpy="${rpy}" />
                 <geometry>
-                    <mesh filename="file:///$(find rob_teleeop)/models/robot_nano_hand_finger1_link${link}.stl" scale="1 1 1"/>
+                    <mesh filename="file:///$(find rob_teleeop)q/robot_nano_hand_finger1_link${link}.stl" scale="1 1 1"/>
                 </geometry>
             </visual>

Commit message: d

File: src/rob_teleeop/rob_teleeop/urdf/finger.urdf.xacro (robot description, xacro)
@@ -6,5 +6,5 @@
                 <origin xyz="${xyz}" rpy="${rpy}" />
                 <geometry>
-                    <mesh filename="file:///$(find rob_teleeop)q/robot_nano_hand_finger1_link${link}.stl" scale="1 1 1"/>
+                    <mesh filename="file:///$(find rob_teleeop)/robot_nano_hand_finger1_link${link}.stl" scale="1 1 1"/>
                 </geometry>
             </visual>

Commit message: qsd

File: src/rob_teleeop/rob_teleeop/urdf/finger.urdf.xacro (robot description, xacro)
@@ -4,5 +4,5 @@
         <link name="${prefix}_link" >
             <visual>
-                <origin xyz="0 0 0" rpy="0 0 0"/>
+                <origin xyz="${xyz}" rpy="${rpy}" />
                 <geometry>
                     <mesh filename="file:///$(find rob_teleeop)/robot_nano_hand_finger1_link${link}.stl" scale="1 1 1"/>

Commit message: qsd

File: src/rob_teleeop/rob_teleeop/urdf/finger.urdf.xacro (robot description, xacro)
@@ -11,5 +11,5 @@
         </link>
         <joint name="${prefix}_joint" type="${joint_type}">
-            <origin xyz="${xyz}" rpy="${rpy}" />
+            <origin xyz="0 0 0" rpy="0 0 0"/>
             <parent link="${parent}"/>
             <child link="${prefix}_link"/>

Commit message: qd

File: src/rob_teleeop/rob_teleeop/urdf/finger.urdf.xacro (robot description, xacro)
@@ -4,5 +4,5 @@
         <link name="${prefix}_link" >
             <visual>
-                <origin xyz="0 0 0" rpy="0 0 1.57"/>
+                <origin xyz="0 0 0" rpy="0 0 0"/>
                 <geometry>
                     <mesh filename="file:///$(find rob_teleeop)/robot_nano_hand_finger1_link${link}.stl" scale="1 1 1"/>

Commit message: qsd

File: src/rob_teleeop/rob_teleeop/urdf/finger.urdf.xacro (robot description, xacro)
@@ -1,5 +1,5 @@
 <?xml version="1.0"?>
 <robot xmlns:xacro="http://ros.org/wiki/xacro" name="finger">
-    <xacro:macro name="finger" params="parent prefix link joint_type xyz rpy a">
+    <xacro:macro name="finger" params="parent prefix link joint_type xyz rpy">
         <link name="${prefix}_link" >
             <visual>

Commit message: qsd

File: src/rob_teleeop/rob_teleeop/urdf/finger.urdf.xacro (robot description, xacro)
@@ -4,5 +4,5 @@
         <link name="${prefix}_link" >
             <visual>
-                <origin xyz="0 0 0" rpy="0 0 1.57"/>
+                <origin xyz="0 0 0" rpy="${-3.14/2} 0 1.57"/>
                 <geometry>
                     <mesh filename="file:///$(find rob_teleeop)/robot_nano_hand_finger1_link${link}.stl" scale="1 1 1"/>

Commit message: qsd

File: src/rob_teleeop/rob_teleeop/urdf/finger.urdf.xacro (robot description, xacro)
@@ -4,5 +4,5 @@
         <link name="${prefix}_link" >
             <visual>
-                <origin xyz="0 0 0" rpy="${-3.14/2} 0 1.57"/>
+                <origin xyz="0 0 0" rpy="0 0 1.57"/>
                 <geometry>
                     <mesh filename="file:///$(find rob_teleeop)/robot_nano_hand_finger1_link${link}.stl" scale="1 1 1"/>

Commit message: qsd

File: src/rob_teleeop/rob_teleeop/urdf/finger.urdf.xacro (robot description, xacro)
@@ -13,4 +13,5 @@
             <origin xyz="${xyz}" rpy="${rpy}" />
             <axis xyz="${axis}"/>
+            <limit effort="0" velocity="0" lower="0" upper="50" />
             <parent link="${parent}"/>
             <child link="${prefix}_link"/>

Commit message: qsdsqd

File: src/rob_teleeop/rob_teleeop/urdf/finger.urdf.xacro (robot description, xacro)
@@ -13,5 +13,5 @@
             <origin xyz="${xyz}" rpy="${rpy}" />
             <axis xyz="${axis}"/>
-            <limit effort="0" velocity="0" lower="0" upper="50" />
+            <limit effort="0" velocity="0" lower="0" upper="1.57" />
             <parent link="${parent}"/>
             <child link="${prefix}_link"/>

Commit message: qsd

File: src/rob_teleeop/rob_teleeop/urdf/finger.urdf.xacro (robot description, xacro)
@@ -13,5 +13,5 @@
             <origin xyz="${xyz}" rpy="${rpy}" />
             <axis xyz="${axis}"/>
-            <limit effort="0" velocity="0" lower="0" upper="1.57" />
+            <limit effort="0" velocity="0" lower="0" upper="0.8" />
             <parent link="${parent}"/>
             <child link="${prefix}_link"/>

Commit message: qsd

File: src/rob_teleeop/rob_teleeop/urdf/finger.urdf.xacro (robot description, xacro)
@@ -13,5 +13,5 @@
             <origin xyz="${xyz}" rpy="${rpy}" />
             <axis xyz="${axis}"/>
-            <limit effort="0" velocity="0" lower="0" upper="0.8" />
+            <limit effort="0" velocity="0" lower="0" upper="0.3" />
             <parent link="${parent}"/>
             <child link="${prefix}_link"/>

Commit message: qsd

File: src/rob_teleeop/rob_teleeop/urdf/finger.urdf.xacro (robot description, xacro)
@@ -13,5 +13,5 @@
             <origin xyz="${xyz}" rpy="${rpy}" />
             <axis xyz="${axis}"/>
-            <limit effort="0" velocity="0" lower="0" upper="0.3" />
+            <limit effort="0" velocity="0" lower="1.57" upper="1.57" />
             <parent link="${parent}"/>
             <child link="${prefix}_link"/>

Commit message: qds

File: src/rob_teleeop/rob_teleeop/urdf/finger.urdf.xacro (robot description, xacro)
@@ -13,5 +13,5 @@
             <origin xyz="${xyz}" rpy="${rpy}" />
             <axis xyz="${axis}"/>
-            <limit effort="0" velocity="0" lower="1.57" upper="1.57" />
+            <limit effort="0" velocity="0" lower="1.57" upper="${1.57+0.5}" />
             <parent link="${parent}"/>
             <child link="${prefix}_link"/>

Commit message: qsd

File: src/rob_teleeop/rob_teleeop/urdf/finger.urdf.xacro (robot description, xacro)
@@ -13,5 +13,5 @@
             <origin xyz="${xyz}" rpy="${rpy}" />
             <axis xyz="${axis}"/>
-            <limit effort="0" velocity="0" lower="1.57" upper="${1.57+0.5}" />
+            <limit effort="0" velocity="0" lower="-100" upper="100" />
             <parent link="${parent}"/>
             <child link="${prefix}_link"/>

Commit message: qsd

File: src/rob_teleeop/rob_teleeop/urdf/finger.urdf.xacro (robot description, xacro)
@@ -1,5 +1,5 @@
 <?xml version="1.0"?>
 <robot xmlns:xacro="http://ros.org/wiki/xacro" name="finger">
-    <xacro:macro name="finger" params="parent nb prefix link joint_type xyz rpy rot axis">
+    <xacro:macro name="finger" params="parent nb link joint_type xyz rpy rot axis">
         <link name="finger${nb}_link{link}" >
             <visual>

Commit message: qsdqsdqsdqsdqsdsd

File: src/rob_teleeop/rob_teleeop/urdf/finger.urdf.xacro (robot description, xacro)
@@ -2,5 +2,5 @@
 <robot xmlns:xacro="http://ros.org/wiki/xacro" name="finger">
     <xacro:macro name="finger" params="parent nb link joint_type xyz rpy rot axis">
-        <link name="finger${nb}_link{link}" >
+        <link name="finger${nb}_link${link}" >
             <visual>
                 <origin xyz="0 0 0" rpy="${rot}"/>
@@ -10,10 +10,10 @@
             </visual>
         </link>
-        <joint name="finger${nb}_joint{link}" type="${joint_type}">
+        <joint name="finger${nb}_joint${link}" type="${joint_type}">
             <origin xyz="${xyz}" rpy="${rpy}" />
             <axis xyz="${axis}"/>
             <limit effort="0" velocity="0" lower="-100" upper="100" />
             <parent link="${parent}"/>
-            <child link="finger${nb}_link{link}"/>
+            <child link="finger${nb}_link${link}"/>
         </joint>
     </xacro:macro>

Commit message: qs

File: src/rob_teleeop/rob_teleeop/urdf/finger.urdf.xacro (robot description, xacro)
@@ -19,5 +19,5 @@
             <origin xyz="${xyz}" rpy="${rpy}" />
             <axis xyz="${axis}"/>
-            <limit effort="0" velocity="0" lower="-100" upper="100" />
+            <limit effort="10" velocity="10" lower="0" upper="1" />
             <parent link="${parent}"/>
             <child link="finger${nb}_link${link}"/>
